File: Hardware/Bus_switch.kicad_sch (KiCad schematic)
At the start: 15 parts, among them J301 Conn_01x04_Pin, U301 SN74CB3Q3384APW

Commit message: finished PCB
Parts:
- removed R301, R302, R303, R307, R309: 10kΩ, PCM_JLCPCB:R_0603, symbol PCM_JLCPCB-Resistors:0603,10kΩ
Other:
- title: MMS3 Hat template small (Change Me) -> MMS3_hat_air_quality
