File: Hardware/MMS3_hat_air_quality.kicad_sch (KiCad schematic)
At the start: 32 parts, among them J101 Conn_01x08, U101 AMS1117, U102 BME688, U103 SCD40-D-R2, U104 BME688, U105 SGP41-D-R4

Commit message: finished readme
Connections:
- net +3V3: now also R103.1
- net GND: no longer R103.1
- net ~{RST}: now reaches J101.6 (Pin_6), R103.2
- net PROTOCOL: now reaches J101.8 (Pin_8), R105.2
- net SET: now reaches J101.3 (Pin_3), R101.1, R102.2, R104.2
- net PWM: now reaches J101.7 (Pin_7)
Other:
- moved on the sheet: J101
Changed lines of the file:
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@@
 	)
 	(no_connect
-		(at 375.92 210.82)
+		(at 374.65 210.82)
 	)
 	(bus_entry
@@
 	(wire
 		(pts
-			(xy 355.6 198.12) (xy 375.92 198.12)
+			(xy 355.6 198.12) (xy 383.54 198.12)
 		)
 		(stroke
@@
 	(wire
 		(pts
-			(xy 337.82 205.74) (xy 375.92 205.74)
+			(xy 337.82 205.74) (xy 383.54 205.74)
 		)
 		(stroke
@@
 	(wire
 		(pts
+			(xy 374.65 210.82) (xy 383.54 210.82)
+		)
+		(stroke
+			(width 0)
+			(type default)
+		)
+	)
+	(wire
+		(pts
 			(xy 326.39 119.38) (xy 331.47 119.38)
 		)
@@
 	(wire
 		(pts
-			(xy 375.92 195.58) (xy 355.6 195.58)
+			(xy 383.54 195.58) (xy 355.6 195.58)
 		)
 		(stroke
@@
 	(wire
 		(pts
-			(xy 312.42 200.66) (xy 375.92 200.66)
+			(xy 312.42 200.66) (xy 383.54 200.66)
 		)
 		(stroke
@@
 	(wire
 		(pts
-			(xy 337.82 203.2) (xy 375.92 203.2)
+			(xy 337.82 203.2) (xy 383.54 203.2)
 		)
 		(stroke
@@
 	(wire
 		(pts
-			(xy 369.57 208.28) (xy 375.92 208.28)
+			(xy 369.57 208.28) (xy 383.54 208.28)
 		)
 		(stroke
@@
 	(wire
 		(pts
-			(xy 369.57 213.36) (xy 375.92 213.36)
+			(xy 369.57 213.36) (xy 383.54 213.36)
 		)
 		(stroke
@@
 		)
 	)
+	(label "~{RST}"
+		(at 377.19 208.28 0)
+		(effects
+			(font
+				(size 1.27 1.27)
+			)
+			(justify left bottom)
+		)
+	)
 	(label "Chainbus.CS"
 		(at 295.91 200.66 180)
@@
 		)
 	)
+	(label "PROTOCOL"
+		(at 373.38 213.36 0)
+		(effects
+			(font
+				(size 1.27 1.27)
+			)
+			(justify left bottom)
+		)
+	)
+	(label "SET"
+		(at 378.46 200.66 0)
+		(effects
+			(font
+				(size 1.27 1.27)
+			)
+			(justify left bottom)
+		)
+	)
 	(label "Chainbus{I2C}"
 		(at 128.27 78.74 180)
@@
 	)
 	(label "Chainbus.TX"
-		(at 369.57 203.2 180)
+		(at 377.19 203.2 180)
 		(effects
 			(font
@@
 	)
 	(label "Chainbus.RX"
-		(at 369.57 205.74 180)
+		(at 377.19 205.74 180)
 		(effects
 			(font
@@
 		)
 	)
+	(label "PWM"
+		(at 377.19 210.82 0)
+		(effects
+			(font
+				(size 1.27 1.27)
+			)
+			(justify left bottom)
+		)
+	)
 	(label "Chainbus.SCL"
 		(at 346.71 134.62 0)
@@
 	(symbol
 		(lib_id "Connector_Generic:Conn_01x08")
-		(at 381 203.2 0)
+		(at 388.62 203.2 0)
 		(unit 1)
 		(body_style 1)
@@
 		(fields_autoplaced yes)
 		(property "Reference" "J101"
-			(at 383.54 203.1999 0)
+			(at 391.16 203.1999 0)
 			(show_name no)
 			(do_not_autoplace no)
@@
 		)
 		(property "Value" "Conn_01x08"
-			(at 383.54 205.7399 0)
+			(at 391.16 205.7399 0)
 			(show_name no)
 			(do_not_autoplace no)
@@
 		)
 		(property "Footprint" "Connector_JST:JST_XH_S8B-XH-A-1_1x08_P2.50mm_Horizontal"
-			(at 381 203.2 0)
+			(at 388.62 203.2 0)
 			(hide yes)
 			(show_name no)
@@
 		)
 		(property "Datasheet" ""
-			(at 381 203.2 0)
+			(at 388.62 203.2 0)
 			(hide yes)
 			(show_name no)
@@
 		)
 		(property "Description" "Generic connector, single row, 01x08, script generated (kicad-library-utils/schlib/autogen/connector/)"
-			(at 381 203.2 0)
+			(at 388.62 203.2 0)
 			(hide yes)
 			(show_name no)
@@
 	)
 	(symbol
-		(lib_id "power:GND")
-		(at 356.87 208.28 270)
-		(unit 1)
-		(body_style 1)
-		(exclude_from_sim no)
-		(in_bom yes)
-		(on_board yes)
-		(in_pos_files yes)
-		(dnp no)
-		(fields_autoplaced yes)
-		(property "Reference" "#PWR0113"
-			(at 350.52 208.28 0)
-			(hide yes)
-			(show_name no)
-			(do_not_autoplace no)
-			(effects
-				(font
-					(size 1.27 1.27)
-				)
-			)
-		)
-		(property "Value" "GND"
-			(at 353.06 208.2799 90)
-			(show_name no)
-			(do_not_autoplace no)
-			(effects
-				(font
-					(size 1.27 1.27)
-				)
-				(justify right)
-			)
-		)
-		(property "Footprint" ""
-			(at 356.87 208.28 0)
-			(hide yes)
-			(show_name no)
-			(do_not_autoplace no)
-			(effects
-				(font
-					(size 1.27 1.27)
-				)
-			)
-		)
-		(property "Datasheet" ""
-			(at 356.87 208.28 0)
-			(hide yes)
-			(show_name no)
-			(do_not_autoplace no)
-			(effects
-				(font
-					(size 1.27 1.27)
-				)
-			)
-		)
-		(property "Description" "Power symbol creates a global label with name \"GND\" , ground"
-			(at 356.87 208.28 0)
-			(hide yes)
-			(show_name no)
-			(do_not_autoplace no)
-			(effects
-				(font
-					(size 1.27 1.27)
-				)
-			)
-		)
-		(pin "1"
-		)
-		(instances
-			(project "MMS3_hat_air_quality"
-				(path "/6596548a-44e0-46d8-8624-fd71cf4a3e17"
-					(reference "#PWR0113")
-					(unit 1)
-				)
-			)
-		)
-	)
-	(symbol
 		(lib_id "PCM_JLCPCB-Resistors:0603,10kΩ")
 		(at 312.42 193.04 0)
@@
 					(unit 1)
 				)
+			)
+		)
+	)
+	(symbol
+		(lib_id "power:+5V")
+		(at 356.87 208.28 90)
+		(mirror x)
+		(unit 1)
+		(body_style 1)
+		(exclude_from_sim no)
+		(in_bom yes)
+		(on_board yes)
+		(in_pos_files yes)
+		(dnp no)
+		(fields_autoplaced yes)
+		(property "Reference" "#PWR0113"
+			(at 360.68 208.28 0)
+			(hide yes)
+			(show_name no)
+			(do_not_autoplace no)
+			(effects
+				(font
+					(size 1.27 1.27)
+				)
+			)
+		)
+		(property "Value" "+3V3"
+			(at 353.06 208.2799 90)
+			(show_name no)
+			(do_not_autoplace no)
+			(effects
+				(font
+					(size 1.27 1.27)
+				)
+				(justify left)
+			)
+		)
+		(property "Footprint" ""
+			(at 356.87 208.28 0)
+			(hide yes)
+			(show_name no)
+			(do_not_autoplace no)
+			(effects
+				(font
+					(size 1.27 1.27)
+				)
+			)
+		)
+		(property "Datasheet" ""
+			(at 356.87 208.28 0)
+			(hide yes)
+			(show_name no)
+			(do_not_autoplace no)
+			(effects
+				(font
+					(size 1.27 1.27)
+				)
+			)
+		)
+		(property "Description" "Power symbol creates a global label with name \"+5V\""
+			(at 356.87 208.28 0)
+			(hide yes)
+			(show_name no)
+			(do_not_autoplace no)
+			(effects
+				(font
+					(size 1.27 1.27)
+				)
+			)
+		)
+		(pin "1"
+		)
+		(instances
+			(project "MMS3_hat_air_quality"
+				(path "/6596548a-44e0-46d8-8624-fd71cf4a3e17"
+					(reference "#PWR0113")
+					(unit 1)
+				)
