File: Hardware/MMS3_hat_air_quality.kicad_pcb (KiCad board)
At the start: 2 copper layers, 100 x 50 mm, 53 parts, among them J101 Conn_01x08, J201 Chainbus in, J202 Chainbus Out, J301 Conn_01x04_Pin, U101 AMS1117, U102 BME688, U103 SCD40-D-R2, U104 BME688, U105 SGP41-D-R4, U301 SN74CB3Q3384APW, U405 ADS1115IDGS, U501 M24C64

Commit message: finished readme
Connections:
- net Net-(J101-Pin_3) renamed /SET
- net Net-(J101-Pin_6) renamed /~{RST}
- net Net-(J101-Pin_8) renamed /PROTOCOL
- J101 pad 7: unconnected-(J101-Pin_7-Pad7) -> /PWM
- R103 pad 1: GND -> +3V3
Routing:
- net +3V3: track 342.0 -> 346.7 mm, vias 22 -> 23
- net GND: track 77.5 -> 76.7 mm, vias 72 -> 71
Changed lines of the file:
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@@
 			(layers "F.Cu" "F.Mask" "F.Paste")
 			(roundrect_rratio 0.25)
-			(net "Net-(J101-Pin_3)")
+			(net "/SET")
 			(pintype "passive")
 		)
@@
 			(layers "F.Cu" "F.Mask" "F.Paste")
 			(roundrect_rratio 0.25)
-			(net "GND")
+			(net "+3V3")
 			(pintype "passive")
 		)
@@
 			(layers "F.Cu" "F.Mask" "F.Paste")
 			(roundrect_rratio 0.25)
-			(net "Net-(J101-Pin_6)")
+			(net "/~{RST}")
 			(pintype "passive")
 		)
@@
 			(layers "*.Cu" "*.Mask")
 			(remove_unused_layers no)
-			(net "Net-(J101-Pin_3)")
+			(net "/SET")
 			(pinfunction "Pin_3_3")
 			(pintype "passive")
@@
 			(layers "*.Cu" "*.Mask")
 			(remove_unused_layers no)
-			(net "Net-(J101-Pin_6)")
+			(net "/~{RST}")
 			(pinfunction "Pin_6_6")
 			(pintype "passive")
@@
 			(layers "*.Cu" "*.Mask")
 			(remove_unused_layers no)
-			(net "unconnected-(J101-Pin_7-Pad7)")
+			(net "/PWM")
 			(pinfunction "Pin_7_7")
 			(pintype "passive+no_connect")
@@
 			(layers "*.Cu" "*.Mask")
 			(remove_unused_layers no)
-			(net "Net-(J101-Pin_8)")
+			(net "/PROTOCOL")
 			(pinfunction "Pin_8_8")
 			(pintype "passive")
@@
 			(layers "F.Cu" "F.Mask" "F.Paste")
 			(roundrect_rratio 0.25)
-			(net "Net-(J101-Pin_3)")
+			(net "/SET")
 			(pintype "passive")
 		)
@@
 			(layers "F.Cu" "F.Mask" "F.Paste")
 			(roundrect_rratio 0.25)
-			(net "Net-(J101-Pin_8)")
+			(net "/PROTOCOL")
 			(pintype "passive")
 		)
@@
 			(layers "F.Cu" "F.Mask" "F.Paste")
 			(roundrect_rratio 0.25)
-			(net "Net-(J101-Pin_3)")
+			(net "/SET")
 			(pintype "passive")
 		)
@@
 	)
 	(segment
-		(start 164.25 122.44)
-		(end 164.25 121.65)
-		(width 0.2)
-		(layer "F.Cu")
-		(net "GND")
-	)
-	(segment
 		(start 111.74 106.8)
 		(end 111.74 105.75)
@@
 		(net "GND")
 	)
-	(via
-		(at 164.25 121.65)
-		(size 0.5)
-		(drill 0.3)
-		(layers "F.Cu" "B.Cu")
-		(net "GND")
-	)
 	(segment
 		(start 143.275 108.5625)
@@
 	)
 	(segment
+		(start 164.25 122.44)
+		(end 164.25 121.65)
+		(width 0.2)
+		(layer "F.Cu")
+		(net "+3V3")
+	)
+	(segment
 		(start 111.74 107.85)
 		(end 111.74 110.53)
@@
 		(net "+3V3")
 	)
+	(via
+		(at 164.25 121.65)
+		(size 0.5)
+		(drill 0.3)
+		(layers "F.Cu" "B.Cu")
+		(net "+3V3")
+	)
 	(segment
 		(start 125.54 128.89)
@@
 	)
 	(segment
+		(start 164.25 121.65)
+		(end 163 122.9)
+		(width 0.2)
+		(layer "B.Cu")
+		(net "+3V3")
+	)
+	(segment
 		(start 139.35 105.7)
 		(end 140.7 107.05)
@@
 	)
 	(segment
+		(start 163 122.9)
+		(end 160.9 122.9)
+		(width 0.2)
+		(layer "B.Cu")
+		(net "+3V3")
+	)
+	(segment
 		(start 141.03 131.22)
 		(end 143.35 131.22)
@@
 	)
 	(segment
-		(start 156.73 123.7)
-		(end 156.73 121.47)
+		(start 177.275 99.505)
+		(end 175.775 99.505)
 		(width 0.2)
 		(layer "F.Cu")
-		(net "Net-(J101-Pin_3)")
+		(net "Net-(D301-Pad1)")
 	)
 	(segment
-		(start 156.73 121.47)
-		(end 156.75 121.45)
+		(start 175.775 99.505)
+		(end 175.77 99.5)
 		(width 0.2)
 		(layer "F.Cu")
-		(net "Net-(J101-Pin_3)")
+		(net "Net-(D301-Pad1)")
 	)
 	(segment
-		(start 156.73 124.17)
-		(end 156.75 124.15)
-		(width 0.2)
+		(start 164.25 136.63)
+		(end 164.23 136.65)
+		(width 0.4)
 		(layer "F.Cu")
-		(net "Net-(J101-Pin_3)")
+		(net "/~{RST}")
 	)
 	(segment
-		(start 156.73 136.65)
-		(end 156.73 124.17)
-		(width 0.2)
+		(start 164.25 124.08)
+		(end 164.25 136.63)
+		(width 0.4)
 		(layer "F.Cu")
-		(net "Net-(J101-Pin_3)")
+		(net "/~{RST}")
 	)
 	(segment
-		(start 156.75 119.67)
-		(end 156.75 121.45)
+		(start 156.73 123.7)
+		(end 156.73 121.47)
 		(width 0.2)
 		(layer "F.Cu")
-		(net "Net-(J101-Pin_3)")
+		(net "/SET")
 	)
 	(segment
-		(start 164.25 136.63)
-		(end 164.23 136.65)
-		(width 0.4)
+		(start 156.73 121.47)
+		(end 156.75 121.45)
+		(width 0.2)
 		(layer "F.Cu")
-		(net "Net-(J101-Pin_6)")
+		(net "/SET")
 	)
 	(segment
-		(start 164.25 124.08)
-		(end 164.25 136.63)
-		(width 0.4)
+		(start 156.73 124.17)
+		(end 156.75 124.15)
+		(width 0.2)
 		(layer "F.Cu")
-		(net "Net-(J101-Pin_6)")
+		(net "/SET")
 	)
 	(segment
-		(start 177.275 99.505)
-		(end 175.775 99.505)
+		(start 156.73 136.65)
+		(end 156.73 124.17)
 		(width 0.2)
 		(layer "F.Cu")
-		(net "Net-(D301-Pad1)")
+		(net "/SET")
 	)
 	(segment
-		(start 175.775 99.505)
-		(end 175.77 99.5)
+		(start 156.75 119.67)
+		(end 156.75 121.45)
 		(width 0.2)
 		(layer "F.Cu")
-		(net "Net-(D301-Pad1)")
+		(net "/SET")
 	)
 	(segment
@@
 		(width 0.4)
 		(layer "F.Cu")
-		(net "Net-(J101-Pin_8)")
+		(net "/PROTOCOL")
 	)
 	(segment
@@
 		(width 0.4)
 		(layer "F.Cu")
-		(net "Net-(J101-Pin_8)")
+		(net "/PROTOCOL")
 	)
 	(zone

Commit message: added I2C Addresses on backsilkscreen
Parts:
- moved G*** 68.2 mm to (167.0, 111.1)
